File: mcu data logger.kicad_sch (KiCad schematic)
At the start: 25 parts, among them U1 24LC1025, U2 DS1337S_, U3 24LC1025, U4 ATMEGA328P-AU, Y1 32.768 KHz, Y2 16 MHz

Commit message: completed board layout
Parts:
- U2: footprint DS1337S_:SOIC127P600X175-8N -> customfootprints:SOIC127P600X175-8N
- U4: footprint (none) -> customfootprints:QFP80P900X900X120-32N
Changed lines of the file:
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@@
 			)
 		)
-		(property "Footprint" " "
+		(property "Footprint" "customfootprints:QFP80P900X900X120-32N"
 			(at 199.136 86.106 0)
 			(effects
@@
 			)
 		)
-		(property "Footprint" "DS1337S_:SOIC127P600X175-8N"
+		(property "Footprint" "customfootprints:SOIC127P600X175-8N"
 			(at 53.34 43.18 0)
 			(effects
